Commit message: edit robot.xacro file

File: xacro/robot.xacro (robot description, xacro)
@@ -4,4 +4,5 @@
 	<xacro:include filename="lrf.xacro" />
 	<xacro:include filename="wheel.xacro" />
+  <!-- =============== Robot base Link & Joint =============== -->
     <link name="base_footprint">
     </link>
@@ -16,5 +17,4 @@
         <visual>
             <geometry>
-                <!--<box size="0.600 0.400 0.050"/>-->
                 <mesh filename="file://$(find kuams_sim)/meshes/KUAMS_ver.5.1.0.dae" />
             </geometry>
@@ -25,5 +25,4 @@
         <collision>
             <geometry>
-                <!--<box size="0.600 0.400 0.050"/>-->
                 <mesh filename="file://$(find kuams_sim)/meshes/KUAMS_ver.5.1.0.dae" />
             </geometry>
@@ -74,17 +73,26 @@
 	<xacro:wheel_macro prefix="frontwheel_right" parent="base_floor" xyz="0.3 0.245 0" rpy="1.57 0 0" axis="0 0 -1" radius="0.1325" length="0.05" mu1="0.0" mu2="1.0"/>
 	<xacro:wheel_macro prefix="frontwheel_left" parent="base_floor" xyz="0.3 -0.245 0" rpy="1.57 0 0" axis="0 0 1" radius="0.1325" length="0.05" mu1="0.0" mu2="1.0"/>
+  <!-- =============== Sensor Link & Joint =============== -->
     <!-- センサーの取り付け位置 -->
-    <link name="sensor_link">
+    <link name="rear_sensor_link">
     </link>
-    <joint name="base_sensor_joint" type="fixed">
+    <joint name="base_rear_sensor_joint" type="fixed">
         <origin rpy="0 0 0" xyz="0.1 0 0.8"/>
         <parent link="base_link"/>
-        <child link="sensor_link"/>
+        <child link="rear_sensor_link"/>
     </joint>
-    <!--LRFの位置-->
-	<!-- <xacro:laser_macro prefix="laser" parent="sensor_arm_link" xyz="0.0 0 0.5" rpy="0 0 0" topic="/scan" visualize="True"/> -->
-    <!-- 3D LRF -->
+    <link name="front_sensor_link">
+    </link>
+    <joint name="base_front_sensor_joint" type="fixed">
+        <origin rpy="3.1415926535 0 0" xyz="0.5 0 0.3"/>
+        <parent link="base_link"/>
+        <child link="front_sensor_link"/>
+    </joint>
+  <!-- =============== Sensors =============== -->
+    <!--LRF-->
+	<xacro:laser_macro prefix="laser" parent="front_sensor_link" xyz="0.0 0 0.0" rpy="0 0 0" topic="/scan" visualize="True"/>
+    <!-- Velodyne VLP-16 -->
     <xacro:include filename="$(find velodyne_description)/urdf/VLP-16.urdf.xacro"/>
-    <xacro:VLP-16 parent="sensor_link" name="velodyne" topic="/velodyne_points" hz="10" samples="440" gpu="true">
+    <xacro:VLP-16 parent="rear_sensor_link" name="velodyne" topic="/velodyne_points" hz="10" samples="440" gpu="true">
         <origin xyz="0.075 0 0.01" rpy="0 0 0" />
     </xacro:VLP-16>
@@ -95,4 +103,5 @@
 		<mu2>0.0</mu2>
 	</gazebo>
+  <!-- =============== Gazebo plugin =============== -->
 	<!--プラグインの設定-->
 	<gazebo>

Commit message: edit xacro file

File: xacro/robot.xacro (robot description, xacro)
@@ -42,24 +42,4 @@
     </joint>
     <link name="footrest_link">
-        <collision>
-            <geometry>
-                <box size="0.250 0.260 0.050"/>
-            </geometry>
-        </collision>
-        <visual>
-            <geometry>
-                <box size="0.250 0.260 0.050"/>
-            </geometry>
-            <material name="grey">
-                <color rgba="0.5 0.5 0.5 1.0"/>
-            </material>
-        </visual>
-        <inertial>
-            <origin xyz="0 0 0" rpy="0 0 0" />
-            <mass value="1" />
-            <inertia ixx="1.0"  ixy="0.0"   ixz="0.0"
-                                iyy="1.0"   iyz="0.0"
-                                            izz="1.0" />
-        </inertial>
     </link>
     <joint name="footrest_joint" type="fixed">
